File: Hardware/AutoLevel Module V2.sch (EAGLE design)
At the start: 11 parts, among them X1 JST-XH-02-PIN-LONG-PAD, X2 JST-XH-02-PIN-LONG-PAD, X3 JST-XH-03-PIN-LONG-PAD

Commit message: RFM V2
Parts:
- removed U$1: SHROOM5MM, RobThePyro:SHROOM5MM
Changed lines of the file:
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@@
 <?xml version="1.0" encoding="utf-8"?>
 <!DOCTYPE eagle SYSTEM "eagle.dtd">
-<eagle version="9.3.0">
+<eagle version="9.3.2">
 <drawing>
 <settings>
@@
 <part name="GND6" library="supply1" deviceset="GND" device=""/>
 <part name="JP5" library="pinhead" deviceset="PINHD-1X1" device=""/>
-<part name="U$1" library="RobThePyro" deviceset="SHROOM" device="5MM"/>
 <part name="U$2" library="RobThePyro" deviceset="SHROOM" device="BOTTOMSILK"/>
 <part name="FRAME1" library="frames" deviceset="FRAME_A_L" device=""/>
@@
 <attribute name="VALUE" x="149.86" y="85.09" size="1.778" layer="96" rot="R270"/>
 </instance>
-<instance part="U$1" gate="G$1" x="177.8" y="35.56" smashed="yes"/>
 <instance part="U$2" gate="G$1" x="167.64" y="35.56" smashed="yes"/>
 <instance part="FRAME1" gate="G$1" x="5.08" y="-33.02" smashed="yes"/>
